File: Amicro_tst.kicad_pcb (KiCad board)
At the start: 2 copper layers, 55.9 x 29 mm, 46 parts, among them J1 Sensor, J2 Progm, J3 Vibr, J4 Pow, J5 Motor out, Q1 Q_NPN_BEC, Q2 Q_NPN_BEC, Q3 Q_NPN_BEC, Q4 Q_NPN_BEC, SW1 RESET, U1 ATmega328-P, U2 24LC512, Y1 Crystal

Commit message: Update Amicro_tst.kicad_pcb
Parts:
- moved J5+ 0.57 mm to (107.6, 126.0)
- renumbered J3 to J3-, J5 to J5+
Routing:
- net VCC: track 104.3 -> 121.1 mm
- net Mt3+: track 0.00 -> 2.08 mm
- net Mt0+: track 0.00 -> 2.08 mm
- net Mt2+: track 0.00 -> 2.07 mm
- net Mt1+: track 0.00 -> 2.07 mm
- net (no net): track 0.00 -> 1.43 mm
Changed lines of the file:
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@@
   )
   (footprint "Connector_PinSocket_1.00mm:PinSocket_1x04_P1.00mm_Vertical" (layer "F.Cu")
-    (at 107.076 126.138 180)
+    (at 107.62 125.9625 180)
     (descr "Through hole straight socket strip, 1x04, 1.00mm pitch, single row (https://gct.co/files/drawings/bc065.pdf), script generated")
     (tags "Through hole socket strip THT 1x04 1.00mm single row")
@@
     (property "Sheetname" "")
     (attr through_hole)
-    (fp_text reference "J5" (at -0.29 -2.027 180) (layer "F.SilkS")
+    (fp_text reference "J5+" (at -0.29 -2.027 180) (layer "F.SilkS")
       (effects (font (size 1 1) (thickness 0.15)))
     )
-    (fp_text value "Motor out" (at -0.29 5.25 180) (layer "F.SilkS")
+    (fp_text value "Motor out" (at 1.72 0.8625 270) (layer "F.SilkS")
       (effects (font (size 0.8 0.8) (thickness 0.15)))
-    )
-    (fp_text user "${REFERENCE}" (at -0.29 1.5 270) (layer "F.Fab")
-      (effects (font (size 0.9 0.9) (thickness 0.14)))
     )
     (fp_line (start 0.52 1.445898) (end 0.52 1.554102) (layer "F.SilkS") (width 0.12))
@@
     (property "Sheetname" "")
     (attr through_hole)
-    (fp_text reference "J3" (at -0.036 -2.032) (layer "F.SilkS")
+    (fp_text reference "J3-" (at -0.036 -2.032) (layer "F.SilkS")
       (effects (font (size 1 1) (thickness 0.15)))
     )
@@
     (property "Sheetname" "")
     (attr smd)
-    (fp_text reference "R10" (at -1.524 -0.004) (layer "B.SilkS")
+    (fp_text reference "R10" (at 0.508 2.792) (layer "B.SilkS")
       (effects (font (size 0.5 0.5) (thickness 0.05)) (justify mirror))
     )
@@
     (property "Sheetname" "")
     (attr smd)
-    (fp_text reference "R11" (at -1.524 -0.004) (layer "B.SilkS")
+    (fp_text reference "R11" (at 0.508 1.774) (layer "B.SilkS")
       (effects (font (size 0.5 0.5) (thickness 0.05)) (justify mirror))
     )
@@
     (property "Sheetname" "")
     (attr smd)
-    (fp_text reference "R8" (at -1.524 0) (layer "B.SilkS")
+    (fp_text reference "R8" (at -2.032 -2.794) (layer "B.SilkS")
       (effects (font (size 0.5 0.5) (thickness 0.05)) (justify mirror))
     )
@@
     (property "Sheetname" "")
     (attr smd)
-    (fp_text reference "R9" (at -1.524 0) (layer "B.SilkS")
+    (fp_text reference "R9" (at 0.508 3.81) (layer "B.SilkS")
       (effects (font (size 0.5 0.5) (thickness 0.05)) (justify mirror))
     )
@@
   )
   (dimension (type aligned) (layer "F.Fab")
-    (pts (xy 105.334 128.956) (xy 160.96 128.956))
+    (pts (xy 105.334 126.416) (xy 160.96 126.416))
     (height 3.556)
-    (gr_text "55.6260 mm" (at 133.147 130.712) (layer "F.Fab")
+    (gr_text "55.6260 mm" (at 133.147 128.172) (layer "F.Fab")
       (effects (font (size 1.5 1.5) (thickness 0.3)))
     )
@@
     (style (thickness 0.15) (arrow_length 1.27) (text_position_mode 0) (extension_height 0.58642) (extension_offset 0.5) keep_text_aligned)
   )
+  (segment (start 156.261 125.019) (end 155.88 125.4) (width 0.2) (layer "F.Cu") (net 0))
+  (segment (start 157.15 125.019) (end 156.261 125.019) (width 0.2) (layer "F.Cu") (net 0))
   (segment (start 125.09 106.731) (end 126.543 106.731) (width 0.4) (layer "F.Cu") (net 1))
   (segment (start 129.464 106.759) (end 129.436 106.731) (width 0.4) (layer "F.Cu") (net 1))
@@
   (segment (start 149.002 106.858) (end 146.482 106.858) (width 0.4) (layer "B.Cu") (net 1))
   (segment (start 114.015094 123.830906) (end 114.015094 121.783622) (width 0.4) (layer "B.Cu") (net 1))
+  (segment (start 110.16 123.04896) (end 110.16 125.4) (width 0.25) (layer "F.Cu") (net 2))
   (segment (start 128.448 111.176) (end 129.464 111.176) (width 0.6) (layer "F.Cu") (net 2))
   (segment (start 129.464 111.176) (end 131.75 108.89) (width 0.6) (layer "F.Cu") (net 2))
   (segment (start 131.75 106.858) (end 131.75 108.89) (width 0.4) (layer "F.Cu") (net 2))
+  (segment (start 110.16 110.414) (end 107.62 112.954) (width 0.4) (layer "F.Cu") (net 2))
+  (segment (start 111.648 122.162) (end 111.04696 122.162) (width 0.25) (layer "F.Cu") (net 2))
+  (segment (start 111.04696 122.162) (end 110.16 123.04896) (width 0.25) (layer "F.Cu") (net 2))
   (segment (start 134.29 104.318) (end 131.75 106.858) (width 0.4) (layer "F.Cu") (net 2))
   (segment (start 142.434 102.742727) (end 140.858727 104.318) (width 0.4) (layer "F.Cu") (net 2))
@@
   (segment (start 127.742604 118.54) (end 128.406 119.203396) (width 0.4) (layer "F.Cu") (net 2))
   (segment (start 144.704 110.668) (end 143.434 111.938) (width 0.6) (layer "F.Cu") (net 2))
+  (segment (start 110.162 126.166) (end 110.162 125.402) (width 0.25) (layer "F.Cu") (net 2))
   (segment (start 143.434 111.938) (end 129.718 111.938) (width 0.6) (layer "F.Cu") (net 2))
   (segment (start 128.448 111.43) (end 128.448 111.176) (width 0.6) (layer "F.Cu") (net 2))
@@
   (segment (start 127.432 111.176) (end 128.448 111.176) (width 0.6) (layer "F.Cu") (net 2))
   (segment (start 133.528 124.638) (end 136.442 124.638) (width 0.4) (layer "F.Cu") (net 2))
+  (segment (start 107.62 118.134) (end 111.648 122.162) (width 0.4) (layer "F.Cu") (net 2))
   (segment (start 140.858727 104.318) (end 134.29 104.318) (width 0.4) (layer "F.Cu") (net 2))
   (segment (start 151.054 119.687) (end 153.594 119.687) (width 0.4) (layer "F.Cu") (net 2))
   (segment (start 129.718 111.938) (end 128.956 111.938) (width 0.6) (layer "F.Cu") (net 2))
-  (segment (start 110.16 110.414) (end 108.092 112.482) (width 0.4) (layer "F.Cu") (net 2))
   (segment (start 154.082 111.938) (end 158.664 116.52) (width 0.6) (layer "F.Cu") (net 2))
   (segment (start 143.434 111.938) (end 154.082 111.938) (width 0.6) (layer "F.Cu") (net 2))
+  (segment (start 107.62 112.954) (end 107.62 118.134) (width 0.4) (layer "F.Cu") (net 2))
   (segment (start 127.686 118.54) (end 127.742604 118.54) (width 0.4) (layer "F.Cu") (net 2))
   (segment (start 142.434 102.576) (end 142.434 102.742727) (width 0.4) (layer "F.Cu") (net 2))
@@
   (via (at 144.704 110.668) (size 0.6) (drill 0.4) (layers "F.Cu" "B.Cu") (net 2))
   (via (at 129.464 111.938) (size 0.6) (drill 0.4) (layers "F.Cu" "B.Cu") (net 2))
+  (segment (start 110.16 125.4) (end 110.16 125.15) (width 0.25) (layer "B.Cu") (net 2))
   (segment (start 129.746 111.966) (end 130.48 111.966) (width 0.4) (layer "B.Cu") (net 2))
+  (segment (start 110.16 125.15) (end 110.162 125.148) (width 0.25) (layer "B.Cu") (net 2))
   (segment (start 129.718 111.938) (end 129.746 111.966) (width 0.4) (layer "B.Cu") (net 2))
   (segment (start 145.464 110.668) (end 144.704 110.668) (width 0.4) (layer "B.Cu") (net 2))
+  (segment (start 110.162 125.402) (end 110.16 125.4) (width 0.25) (layer "B.Cu") (net 2))
   (segment (start 146.99 108.89) (end 145.466 107.366) (width 0.3) (layer "F.Cu") (net 3))
   (segment (start 141.734 107.19) (end 141.734 105.334) (width 0.3) (layer "F.Cu") (net 3))
@@
   (segment (start 116.51 106.096) (end 116.51 108.89) (width 0.4) (layer "F.Cu") (net 34))
   (segment (start 113.97 106.096) (end 113.97 108.89) (width 0.4) (layer "F.Cu") (net 35))
+  (segment (start 107.104 126.166) (end 107.076 126.138) (width 0.25) (layer "B.Cu") (net 36))
+  (segment (start 109.142 126.166) (end 107.104 126.166) (width 0.25) (layer "B.Cu") (net 36))
+  (segment (start 107.086 125.148) (end 107.076 125.138) (width 0.25) (layer "B.Cu") (net 37))
+  (segment (start 109.142 125.148) (end 107.086 125.148) (width 0.25) (layer "B.Cu") (net 37))
+  (segment (start 109.142 124.13) (end 107.084 124.13) (width 0.25) (layer "B.Cu") (net 38))
+  (segment (start 107.084 124.13) (end 107.076 124.138) (width 0.25) (layer "B.Cu") (net 38))
+  (segment (start 107.1 123.114) (end 107.076 123.138) (width 0.25) (layer "B.Cu") (net 39))
+  (segment (start 109.142 123.114) (end 107.1 123.114) (width 0.25) (layer "B.Cu") (net 39))
 )
