File: Amicro_tst.kicad_pcb (KiCad board)
At the start: 2 copper layers, 55.9 x 29 mm, 46 parts, among them J1 Sensor, J2 Progm, J3- Vibr, J4 Pow, J5+ Motor out, Q1 Q_NPN_BEC, Q2 Q_NPN_BEC, Q3 Q_NPN_BEC, Q4 Q_NPN_BEC, SW1 RESET, U1 ATmega328-P, U2 24LC512, Y1 Crystal

Commit message: changed board/schem issue and Gerber/cad
Parts:
- J5: renamed from J5+; value Motor out -> Motor Pow
- moved J3 0.29 mm to (111.9, 126.2)
- moved J5 0.29 mm to (107.9, 126.0)
- moved R10 0.29 mm to (109.9, 125.1)
- moved R11 0.29 mm to (109.9, 126.2)
- moved R8 0.29 mm to (109.9, 123.1)
- moved R9 0.29 mm to (109.9, 124.1)
- renumbered J3- to J3, TP(12)1 to TP(12), TP(13)1 to TP(13), TP(14)1 to TP(14), TP(24)1 to TP(24), TP(25)1 to TP(25), TP(26)1 to TP(26), TP(4)1 to TP(4), TP(6)1 to TP(6), TP(7)1 to TP(7)
Routing:
- net (no net): track 1.43 -> 0.00 mm
- net M2: track 17.3 -> 16.7 mm

Commit message: Updated Gerbers
Parts:
- R1: value 50 -> 1k
- moved D1 0.25 mm to (125.1, 119.3)
- renumbered J3 to J3-, J5 to J5+
Connections:
- R1 pad 1: VCC -> GND
Routing:
- net GND: track 148.5 -> 153.0 mm, vias 1 -> 2
