File: Amicro_tst.kicad_sch (KiCad schematic)
At the start: 44 parts, among them J1 Sensor, J2 Progm, J3 Vibr, J4 Pow, J5 Conn_01x04_Female, Q1 Q_NPN_BEC, Q2 Q_NPN_BEC, Q3 Q_NPN_BEC, Q4 Q_NPN_BEC, SW1 RESET, U1 ATmega328-P, U2 24LC512, Y1 Crystal

Commit message: changed board/schem issue and Gerber/cad
Parts:
- J5+: renamed from J5; value Conn_01x04_Female -> Motor Pow
- TP(19): renamed from TP(19)1; value TestPoint -> TP; footprint (none) -> TestPoint:TestPoint_THTPad_1.0x1.0mm_Drill0.5mm
- renumbered J3 to J3-, TP(12)1 to TP(12), TP(13)1 to TP(13), TP(14)1 to TP(14), TP(24)1 to TP(24), TP(25)1 to TP(25), TP(26)1 to TP(26), TP(4)1 to TP(4), TP(6)1 to TP(6), TP(7)1 to TP(7)
Changed lines of the file:
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@@
   (symbol (lib_id "Connector:TestPoint_Small") (at 67.31 149.86 270) (unit 1)
     (in_bom yes) (on_board yes)
-    (property "Reference" "TP(13)1" (id 0) (at 68.5801 151.13 0)
+    (property "Reference" "TP(13)" (id 0) (at 68.5801 151.13 0)
       (effects (font (size 1.27 1.27)) (justify left))
     )
@@
   (symbol (lib_id "Connector:TestPoint_Small") (at 72.39 77.47 0) (unit 1)
     (in_bom yes) (on_board yes)
-    (property "Reference" "TP(14)1" (id 0) (at 73.66 76.1999 0)
+    (property "Reference" "TP(14)" (id 0) (at 73.66 76.1999 0)
       (effects (font (size 1.27 1.27)) (justify left))
     )
@@
   (symbol (lib_id "Connector:TestPoint_Small") (at 74.93 149.86 270) (unit 1)
     (in_bom yes) (on_board yes)
-    (property "Reference" "TP(12)1" (id 0) (at 76.2001 151.13 0)
+    (property "Reference" "TP(12)" (id 0) (at 76.2001 151.13 0)
       (effects (font (size 1.27 1.27)) (justify left))
     )
@@
   (symbol (lib_id "Connector:TestPoint_Small") (at 86.36 111.76 0) (unit 1)
     (in_bom yes) (on_board yes)
-    (property "Reference" "TP(25)1" (id 0) (at 87.63 110.4899 0)
+    (property "Reference" "TP(25)" (id 0) (at 87.63 110.4899 0)
       (effects (font (size 1.27 1.27)) (justify left))
     )
@@
   (symbol (lib_id "Connector:TestPoint_Small") (at 93.98 144.78 0) (unit 1)
     (in_bom yes) (on_board yes)
-    (property "Reference" "TP(6)1" (id 0) (at 95.25 143.5099 0)
+    (property "Reference" "TP(6)" (id 0) (at 95.25 143.5099 0)
       (effects (font (size 1.27 1.27)) (justify left))
     )
@@
   (symbol (lib_id "Connector:TestPoint_Small") (at 88.9 133.35 0) (unit 1)
     (in_bom yes) (on_board yes)
-    (property "Reference" "TP(4)1" (id 0) (at 90.17 132.0799 0)
+    (property "Reference" "TP(4)" (id 0) (at 90.17 132.0799 0)
       (effects (font (size 1.27 1.27)) (justify left))
     )
@@
   (symbol (lib_id "Connector:TestPoint") (at 102.87 80.01 0) (unit 1)
     (in_bom yes) (on_board yes) (fields_autoplaced)
-    (property "Reference" "TP(19)1" (id 0) (at 105.41 75.4379 0)
-      (effects (font (size 1.27 1.27)) (justify left))
-    )
-    (property "Value" "TestPoint" (id 1) (at 105.41 77.9779 0)
-      (effects (font (size 1.27 1.27)) (justify left))
-    )
-    (property "Footprint" "" (id 2) (at 107.95 80.01 0)
+    (property "Reference" "TP(19)" (id 0) (at 105.41 75.4379 0)
+      (effects (font (size 1.27 1.27)) (justify left))
+    )
+    (property "Value" "TP" (id 1) (at 105.41 77.9779 0)
+      (effects (font (size 1.27 1.27)) (justify left))
+    )
+    (property "Footprint" "TestPoint:TestPoint_THTPad_1.0x1.0mm_Drill0.5mm" (id 2) (at 107.95 80.01 0)
       (effects (font (size 1.27 1.27)) hide)
     )
@@
   (symbol (lib_id "Connector:TestPoint_Small") (at 85.09 106.68 0) (unit 1)
     (in_bom yes) (on_board yes)
-    (property "Reference" "TP(24)1" (id 0) (at 86.36 105.4099 0)
+    (property "Reference" "TP(24)" (id 0) (at 86.36 105.4099 0)
       (effects (font (size 1.27 1.27)) (justify left))
     )
@@
   (symbol (lib_id "Connector:Conn_01x04_Female") (at 215.9 152.4 0) (unit 1)
     (in_bom yes) (on_board yes) (fields_autoplaced)
-    (property "Reference" "J5" (id 0) (at 217.17 152.3999 0)
-      (effects (font (size 1.27 1.27)) (justify left))
-    )
-    (property "Value" "Conn_01x04_Female" (id 1) (at 217.17 154.9399 0)
+    (property "Reference" "J5+" (id 0) (at 217.17 152.3999 0)
+      (effects (font (size 1.27 1.27)) (justify left))
+    )
+    (property "Value" "Motor Pow" (id 1) (at 217.17 154.9399 0)
       (effects (font (size 1.27 1.27)) (justify left))
     )
@@
   (symbol (lib_id "Connector:TestPoint_Small") (at 86.36 116.84 0) (unit 1)
     (in_bom yes) (on_board yes)
-    (property "Reference" "TP(26)1" (id 0) (at 87.63 115.5699 0)
+    (property "Reference" "TP(26)" (id 0) (at 87.63 115.5699 0)
       (effects (font (size 1.27 1.27)) (justify left))
     )
@@
   (symbol (lib_id "Connector:Conn_01x05_Female") (at 273.05 115.57 0) (unit 1)
     (in_bom yes) (on_board yes) (fields_autoplaced)
-    (property "Reference" "J3" (id 0) (at 274.32 114.2999 0)
+    (property "Reference" "J3-" (id 0) (at 274.32 114.2999 0)
       (effects (font (size 1.27 1.27)) (justify left))
     )
@@
   (symbol (lib_id "Connector:TestPoint_Small") (at 88.9 138.43 0) (unit 1)
     (in_bom yes) (on_board yes)
-    (property "Reference" "TP(7)1" (id 0) (at 90.17 137.1599 0)
+    (property "Reference" "TP(7)" (id 0) (at 90.17 137.1599 0)
       (effects (font (size 1.27 1.27)) (justify left))
     )
@@
     )
     (path "/d06bff60-dd66-4461-a791-89966a79340a"
-      (reference "J3") (unit 1) (value "Vibr") (footprint "Connector_PinSocket_1.00mm:PinSocket_1x05_P1.00mm_Vertical")
+      (reference "J3-") (unit 1) (value "Vibr") (footprint "Connector_PinSocket_1.00mm:PinSocket_1x05_P1.00mm_Vertical")
     )
     (path "/b3060f11-28e1-4ef4-8cb3-348282790846"
@@
     )
     (path "/b4ffede1-34cd-4565-b296-e6cffdffcf56"
-      (reference "J5") (unit 1) (value "Conn_01x04_Female") (footprint "Connector_PinSocket_1.00mm:PinSocket_1x04_P1.00mm_Vertical")
+      (reference "J5+") (unit 1) (value "Motor Pow") (footprint "Connector_PinSocket_1.00mm:PinSocket_1x04_P1.00mm_Vertical")
     )
     (path "/9151b024-63a6-41bc-be59-5e0747a6c69f"
@@
     )
     (path "/57803f16-4951-4322-937a-3335afb08842"
-      (reference "TP(4)1") (unit 1) (value "TP") (footprint "TestPoint:TestPoint_THTPad_1.0x1.0mm_Drill0.5mm")
+      (reference "TP(4)") (unit 1) (value "TP") (footprint "TestPoint:TestPoint_THTPad_1.0x1.0mm_Drill0.5mm")
     )
     (path "/463e4c84-30ed-487f-958a-8d35a40efe38"
-      (reference "TP(6)1") (unit 1) (value "TP") (footprint "TestPoint:TestPoint_THTPad_1.0x1.0mm_Drill0.5mm")
+      (reference "TP(6)") (unit 1) (value "TP") (footprint "TestPoint:TestPoint_THTPad_1.0x1.0mm_Drill0.5mm")
     )
     (path "/d747968d-1725-40a5-bf12-3208d9131768"
-      (reference "TP(7)1") (unit 1) (value "TP") (footprint "TestPoint:TestPoint_THTPad_1.0x1.0mm_Drill0.5mm")
+      (reference "TP(7)") (unit 1) (value "TP") (footprint "TestPoint:TestPoint_THTPad_1.0x1.0mm_Drill0.5mm")
     )
     (path "/3afe24a8-dc8f-418b-8ea7-f4d6e4f519c6"
-      (reference "TP(12)1") (unit 1) (value "TP") (footprint "TestPoint:TestPoint_THTPad_1.0x1.0mm_Drill0.5mm")
+      (reference "TP(12)") (unit 1) (value "TP") (footprint "TestPoint:TestPoint_THTPad_1.0x1.0mm_Drill0.5mm")
     )
     (path "/05ab7aa5-7b8e-4104-a8d0-893eabc178ac"
-      (reference "TP(13)1") (unit 1) (value "TP") (footprint "TestPoint:TestPoint_THTPad_1.0x1.0mm_Drill0.5mm")
+      (reference "TP(13)") (unit 1) (value "TP") (footprint "TestPoint:TestPoint_THTPad_1.0x1.0mm_Drill0.5mm")
     )
     (path "/1e8636dc-257b-4ddd-a4ee-08d597e947fe"
-      (reference "TP(14)1") (unit 1) (value "TP") (footprint "TestPoint:TestPoint_THTPad_1.0x1.0mm_Drill0.5mm")
+      (reference "TP(14)") (unit 1) (value "TP") (footprint "TestPoint:TestPoint_THTPad_1.0x1.0mm_Drill0.5mm")
     )
     (path "/654beb0c-1bb6-4ccb-9b7c-c689f185edc1"
-      (reference "TP(19)1") (unit 1) (value "TestPoint") (footprint "")
+      (reference "TP(19)") (unit 1) (value "TP") (footprint "TestPoint:TestPoint_THTPad_1.0x1.0mm_Drill0.5mm")
     )
     (path "/8ca58ff6-3d0e-4962-8f97-a2d132bb9ca5"
-      (reference "TP(24)1") (unit 1) (value "TP") (footprint "TestPoint:TestPoint_THTPad_1.0x1.0mm_Drill0.5mm")
+      (reference "TP(24)") (unit 1) (value "TP") (footprint "TestPoint:TestPoint_THTPad_1.0x1.0mm_Drill0.5mm")
     )
     (path "/3be7a91a-0e4e-4700-b7a6-05629a300185"
-      (reference "TP(25)1") (unit 1) (value "TP") (footprint "TestPoint:TestPoint_THTPad_1.0x1.0mm_Drill0.5mm")
+      (reference "TP(25)") (unit 1) (value "TP") (footprint "TestPoint:TestPoint_THTPad_1.0x1.0mm_Drill0.5mm")
     )
     (path "/bfc17877-a75d-4438-bd98-4babebb460e0"
-      (reference "TP(26)1") (unit 1) (value "TP") (footprint "TestPoint:TestPoint_THTPad_1.0x1.0mm_Drill0.5mm")
+      (reference "TP(26)") (unit 1) (value "TP") (footprint "TestPoint:TestPoint_THTPad_1.0x1.0mm_Drill0.5mm")
     )
     (path "/6edf16be-7bba-4219-b66e-987d0571c267"

Commit message: Updated Gerbers
Parts:
- R1: value 50 -> 1k
Changed lines of the file:
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@@
       (effects (font (size 1.27 1.27)) (justify left))
     )
-    (property "Value" "50" (id 1) (at 97.79 82.5499 0)
+    (property "Value" "1k" (id 1) (at 97.79 82.5499 0)
       (effects (font (size 1.27 1.27)) (justify left))
     )
@@
     )
     (path "/2719589e-6f3e-41f2-ae58-0c107b009320"
-      (reference "R1") (unit 1) (value "50") (footprint "Resistor_SMD:R_0402_1005Metric")
+      (reference "R1") (unit 1) (value "1k") (footprint "Resistor_SMD:R_0402_1005Metric")
     )
     (path "/bc02e175-2ba0-4b50-83cf-01e6a8d434ed"

Commit message: .
Parts:
- renumbered J3- to J3-1, J5+ to J5+1, TP(12) to TP(12)1, TP(13) to TP(13)1, TP(14) to TP(14)1, TP(19) to TP(19)1, TP(24) to TP(24)1, TP(25) to TP(25)1, TP(26) to TP(26)1, TP(4) to TP(4)1, TP(6) to TP(6)1, TP(7) to TP(7)1
Connections:
- net GND: now also R1.1
- net VCC: no longer R1.1
Changed lines of the file:
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@@
+    (stroke (width 0) (type default) (color 0 0 0 0))
+  )
+  (wire (pts (xy 88.9 72.39) (xy 95.25 72.39))
     (stroke (width 0) (type default) (color 0 0 0 0))
   )
@@
     (stroke (width 0) (type default) (color 0 0 0 0))
   )
-  (wire (pts (xy 95.25 73.66) (xy 95.25 74.93))
+  (wire (pts (xy 95.25 72.39) (xy 95.25 74.93))
     (stroke (width 0) (type default) (color 0 0 0 0))
   )
@@
   (symbol (lib_id "Connector:TestPoint_Small") (at 67.31 149.86 270) (unit 1)
     (in_bom yes) (on_board yes)
-    (property "Reference" "TP(13)" (id 0) (at 68.5801 151.13 0)
+    (property "Reference" "TP(13)1" (id 0) (at 68.5801 151.13 0)
       (effects (font (size 1.27 1.27)) (justify left))
     )
@@
   (symbol (lib_id "Connector:TestPoint_Small") (at 72.39 77.47 0) (unit 1)
     (in_bom yes) (on_board yes)
-    (property "Reference" "TP(14)" (id 0) (at 73.66 76.1999 0)
+    (property "Reference" "TP(14)1" (id 0) (at 73.66 76.1999 0)
       (effects (font (size 1.27 1.27)) (justify left))
     )
@@
   (symbol (lib_id "Connector:TestPoint_Small") (at 74.93 149.86 270) (unit 1)
     (in_bom yes) (on_board yes)
-    (property "Reference" "TP(12)" (id 0) (at 76.2001 151.13 0)
+    (property "Reference" "TP(12)1" (id 0) (at 76.2001 151.13 0)
       (effects (font (size 1.27 1.27)) (justify left))
     )
@@
   (symbol (lib_id "Connector:TestPoint_Small") (at 86.36 111.76 0) (unit 1)
     (in_bom yes) (on_board yes)
-    (property "Reference" "TP(25)" (id 0) (at 87.63 110.4899 0)
+    (property "Reference" "TP(25)1" (id 0) (at 87.63 110.4899 0)
       (effects (font (size 1.27 1.27)) (justify left))
     )
@@
   (symbol (lib_id "Connector:TestPoint_Small") (at 93.98 144.78 0) (unit 1)
     (in_bom yes) (on_board yes)
-    (property "Reference" "TP(6)" (id 0) (at 95.25 143.5099 0)
+    (property "Reference" "TP(6)1" (id 0) (at 95.25 143.5099 0)
       (effects (font (size 1.27 1.27)) (justify left))
     )
@@
   (symbol (lib_id "Connector:TestPoint_Small") (at 88.9 133.35 0) (unit 1)
     (in_bom yes) (on_board yes)
-    (property "Reference" "TP(4)" (id 0) (at 90.17 132.0799 0)
+    (property "Reference" "TP(4)1" (id 0) (at 90.17 132.0799 0)
       (effects (font (size 1.27 1.27)) (justify left))
     )
@@
   (symbol (lib_id "Connector:TestPoint") (at 102.87 80.01 0) (unit 1)
     (in_bom yes) (on_board yes) (fields_autoplaced)
-    (property "Reference" "TP(19)" (id 0) (at 105.41 75.4379 0)
+    (property "Reference" "TP(19)1" (id 0) (at 105.41 75.4379 0)
       (effects (font (size 1.27 1.27)) (justify left))
     )
@@
   (symbol (lib_id "Connector:TestPoint_Small") (at 85.09 106.68 0) (unit 1)
     (in_bom yes) (on_board yes)
-    (property "Reference" "TP(24)" (id 0) (at 86.36 105.4099 0)
+    (property "Reference" "TP(24)1" (id 0) (at 86.36 105.4099 0)
       (effects (font (size 1.27 1.27)) (justify left))
     )
@@
     (pin "2")
   )
+  (symbol (lib_id "power:GND") (at 88.9 72.39 0) (unit 1)
+    (in_bom yes) (on_board yes) (fields_autoplaced)
+    (property "Reference" "#PWR0112" (id 0) (at 88.9 78.74 0)
+      (effects (font (size 1.27 1.27)) hide)
+    )
+    (property "Value" "GND" (id 1) (at 88.9 77.47 0))
+    (property "Footprint" "" (id 2) (at 88.9 72.39 0)
+      (effects (font (size 1.27 1.27)) hide)
+    )
+    (property "Datasheet" "" (id 3) (at 88.9 72.39 0)
+      (effects (font (size 1.27 1.27)) hide)
+    )
+    (pin "1")
+  )
   (symbol (lib_id "Device:R") (at 233.68 83.82 90) (unit 1)
     (in_bom yes) (on_board yes) (fields_autoplaced)
@@
   (symbol (lib_id "Connector:Conn_01x04_Female") (at 215.9 152.4 0) (unit 1)
     (in_bom yes) (on_board yes) (fields_autoplaced)
-    (property "Reference" "J5+" (id 0) (at 217.17 152.3999 0)
+    (property "Reference" "J5+1" (id 0) (at 217.17 152.3999 0)
       (effects (font (size 1.27 1.27)) (justify left))
     )
@@
   (symbol (lib_id "Connector:TestPoint_Small") (at 86.36 116.84 0) (unit 1)
     (in_bom yes) (on_board yes)
-    (property "Reference" "TP(26)" (id 0) (at 87.63 115.5699 0)
+    (property "Reference" "TP(26)1" (id 0) (at 87.63 115.5699 0)
       (effects (font (size 1.27 1.27)) (justify left))
     )
@@
   (symbol (lib_id "Connector:Conn_01x05_Female") (at 273.05 115.57 0) (unit 1)
     (in_bom yes) (on_board yes) (fields_autoplaced)
-    (property "Reference" "J3-" (id 0) (at 274.32 114.2999 0)
+    (property "Reference" "J3-1" (id 0) (at 274.32 114.2999 0)
       (effects (font (size 1.27 1.27)) (justify left))
     )
@@
   (symbol (lib_id "Connector:TestPoint_Small") (at 88.9 138.43 0) (unit 1)
     (in_bom yes) (on_board yes)
-    (property "Reference" "TP(7)" (id 0) (at 90.17 137.1599 0)
+    (property "Reference" "TP(7)1" (id 0) (at 90.17 137.1599 0)
       (effects (font (size 1.27 1.27)) (justify left))
     )
@@
     (pin "2")
   )
-  (symbol (lib_id "power:VCC") (at 95.25 73.66 0) (unit 1)
-    (in_bom yes) (on_board yes)
-    (property "Reference" "#PWR0112" (id 0) (at 95.25 77.47 0)
-      (effects (font (size 1.27 1.27)) hide)
-    )
-    (property "Value" "VCC" (id 1) (at 95.25 68.58 0))
-    (property "Footprint" "" (id 2) (at 95.25 73.66 0)
-      (effects (font (size 1.27 1.27)) hide)
-    )
-    (property "Datasheet" "" (id 3) (at 95.25 73.66 0)
-      (effects (font (size 1.27 1.27)) hide)
-    )
-    (pin "1")
-  )
   (symbol (lib_id "Device:LED") (at 83.82 87.63 180) (unit 1)
     (in_bom yes) (on_board yes) (fields_autoplaced)
@@
       (reference "#PWR0111") (unit 1) (value "VCC") (footprint "")
     )
-    (path "/dfda7cbd-bb51-487d-89df-dcc6474ce38e"
-      (reference "#PWR0112") (unit 1) (value "VCC") (footprint "")
+    (path "/959a9413-2185-4741-8815-068ada47cddc"
+      (reference "#PWR0112") (unit 1) (value "GND") (footprint "")
     )
     (path "/ba302119-714b-4f33-b283-8c837c71a401"
@@
     )
     (path "/d06bff60-dd66-4461-a791-89966a79340a"
-      (reference "J3-") (unit 1) (value "Vibr") (footprint "Connector_PinSocket_1.00mm:PinSocket_1x05_P1.00mm_Vertical")
+      (reference "J3-1") (unit 1) (value "Vibr") (footprint "Connector_PinSocket_1.00mm:PinSocket_1x05_P1.00mm_Vertical")
     )
     (path "/b3060f11-28e1-4ef4-8cb3-348282790846"
@@
     )
     (path "/b4ffede1-34cd-4565-b296-e6cffdffcf56"
-      (reference "J5+") (unit 1) (value "Motor Pow") (footprint "Connector_PinSocket_1.00mm:PinSocket_1x04_P1.00mm_Vertical")
+      (reference "J5+1") (unit 1) (value "Motor Pow") (footprint "Connector_PinSocket_1.00mm:PinSocket_1x04_P1.00mm_Vertical")
     )
     (path "/9151b024-63a6-41bc-be59-5e0747a6c69f"
@@
     )
     (path "/57803f16-4951-4322-937a-3335afb08842"
-      (reference "TP(4)") (unit 1) (value "TP") (footprint "TestPoint:TestPoint_THTPad_1.0x1.0mm_Drill0.5mm")
+      (reference "TP(4)1") (unit 1) (value "TP") (footprint "TestPoint:TestPoint_THTPad_1.0x1.0mm_Drill0.5mm")
     )
     (path "/463e4c84-30ed-487f-958a-8d35a40efe38"
-      (reference "TP(6)") (unit 1) (value "TP") (footprint "TestPoint:TestPoint_THTPad_1.0x1.0mm_Drill0.5mm")
+      (reference "TP(6)1") (unit 1) (value "TP") (footprint "TestPoint:TestPoint_THTPad_1.0x1.0mm_Drill0.5mm")
     )
     (path "/d747968d-1725-40a5-bf12-3208d9131768"
-      (reference "TP(7)") (unit 1) (value "TP") (footprint "TestPoint:TestPoint_THTPad_1.0x1.0mm_Drill0.5mm")
+      (reference "TP(7)1") (unit 1) (value "TP") (footprint "TestPoint:TestPoint_THTPad_1.0x1.0mm_Drill0.5mm")
     )
     (path "/3afe24a8-dc8f-418b-8ea7-f4d6e4f519c6"
-      (reference "TP(12)") (unit 1) (value "TP") (footprint "TestPoint:TestPoint_THTPad_1.0x1.0mm_Drill0.5mm")
+      (reference "TP(12)1") (unit 1) (value "TP") (footprint "TestPoint:TestPoint_THTPad_1.0x1.0mm_Drill0.5mm")
     )
     (path "/05ab7aa5-7b8e-4104-a8d0-893eabc178ac"
-      (reference "TP(13)") (unit 1) (value "TP") (footprint "TestPoint:TestPoint_THTPad_1.0x1.0mm_Drill0.5mm")
+      (reference "TP(13)1") (unit 1) (value "TP") (footprint "TestPoint:TestPoint_THTPad_1.0x1.0mm_Drill0.5mm")
     )
     (path "/1e8636dc-257b-4ddd-a4ee-08d597e947fe"
-      (reference "TP(14)") (unit 1) (value "TP") (footprint "TestPoint:TestPoint_THTPad_1.0x1.0mm_Drill0.5mm")
+      (reference "TP(14)1") (unit 1) (value "TP") (footprint "TestPoint:TestPoint_THTPad_1.0x1.0mm_Drill0.5mm")
     )
     (path "/654beb0c-1bb6-4ccb-9b7c-c689f185edc1"
-      (reference "TP(19)") (unit 1) (value "TP") (footprint "TestPoint:TestPoint_THTPad_1.0x1.0mm_Drill0.5mm")
+      (reference "TP(19)1") (unit 1) (value "TP") (footprint "TestPoint:TestPoint_THTPad_1.0x1.0mm_Drill0.5mm")
     )
     (path "/8ca58ff6-3d0e-4962-8f97-a2d132bb9ca5"
-      (reference "TP(24)") (unit 1) (value "TP") (footprint "TestPoint:TestPoint_THTPad_1.0x1.0mm_Drill0.5mm")
+      (reference "TP(24)1") (unit 1) (value "TP") (footprint "TestPoint:TestPoint_THTPad_1.0x1.0mm_Drill0.5mm")
     )
     (path "/3be7a91a-0e4e-4700-b7a6-05629a300185"
-      (reference "TP(25)") (unit 1) (value "TP") (footprint "TestPoint:TestPoint_THTPad_1.0x1.0mm_Drill0.5mm")
+      (reference "TP(25)1") (unit 1) (value "TP") (footprint "TestPoint:TestPoint_THTPad_1.0x1.0mm_Drill0.5mm")
     )
     (path "/bfc17877-a75d-4438-bd98-4babebb460e0"
-      (reference "TP(26)") (unit 1) (value "TP") (footprint "TestPoint:TestPoint_THTPad_1.0x1.0mm_Drill0.5mm")
+      (reference "TP(26)1") (unit 1) (value "TP") (footprint "TestPoint:TestPoint_THTPad_1.0x1.0mm_Drill0.5mm")
     )
     (path "/6edf16be-7bba-4219-b66e-987d0571c267"
